File: catt_sao.kicad_pcb (KiCad board)
At the start: 2 copper layers, 20 x 20 mm, 2 parts, among them J1 CATT, J2 SAO

Commit message: Version 2
Parts:
- added J3: SAO, Connector_PinSocket_2.54mm:PinSocket_2x03_P2.54mm_Vertical, F.Cu at (-7.46, 7.62)
- moved J2 7.81 mm to (-12.5, -7.62)
Connections:
- J1 pad 10: SAO_IO1 -> SAO_IO1a
- J1 pad 2: P4_RESET -> unconnected-(J1-Pin_2-Pad2)
- J1 pad 5: MTDI -> unconnected-(J1-Pin_5-Pad5)
- J1 pad 6: MTCK -> unconnected-(J1-Pin_6-Pad6)
- J1 pad 7: MTDO -> SAO_IO2b
- J1 pad 8: MTMS -> SAO_IO1b
- J1 pad 9: SAO_IO2 -> SAO_IO2a
- J2 pad 5: SAO_IO1 -> SAO_IO1b
- J2 pad 6: SAO_IO2 -> SAO_IO2b
Routing:
- net SAO_IO1a: track 0.00 -> 24.1 mm
- net SAO_IO1b: track 0.00 -> 19.2 mm
- net SAO_IO2a: track 0.00 -> 18.8 mm, vias 0 -> 1
- net SAO_SDA: track 15.0 -> 33.3 mm
- net SAO_IO2b: track 0.00 -> 17.0 mm
- net +3.3V: track 37.2 -> 53.8 mm
- net SAO_SCL: track 12.4 -> 24.6 mm
- net SAO_IO1: track 12.0 -> 0.00 mm
- net SAO_IO2: track 7.40 -> 0.00 mm
- net GND: vias 3 -> 0
- removed copper zone on B.Cu, net GND
Other:
- board size 20 x 20 mm -> 24 x 20 mm
- board text added: "Nicolai Electronics"
- board text added: "SAO"
- board text added: "SAO to CATT adapter"
- board text added: "This side should face the back of the device"
- board text removed: "CATT SAO"
- board text removed: "This side should face to the back of the device"
