File: catt_sao.kicad_sch (KiCad schematic)
At the start: 2 parts, among them J1 CATT, J2 SAO

Commit message: Version 2
Parts:
- added J3: SAO, Connector_PinSocket_2.54mm:PinSocket_2x03_P2.54mm_Vertical, symbol Connector_Generic:Conn_02x03_Odd_Even
Connections:
- net +3.3V: now also J3.1 (Pin_1)
- net GND: now also J3.2 (Pin_2)
- net SAO_SCL: now also J3.4 (Pin_4)
- net SAO_SDA: now also J3.3 (Pin_3)
- net MTCK: no longer names the net of J1.6 (Pin_6)
- net MTDI: no longer names the net of J1.5 (Pin_5)
- net MTDO renamed SAO_IO2b
- net SAO_IO2b: now also J2.6 (Pin_6)
- net MTMS renamed SAO_IO1b
- net SAO_IO1b: now also J2.5 (Pin_5)
- net P4_RESET: no longer names the net of J1.2 (Pin_2)
- net SAO_IO1 renamed SAO_IO1a
- net SAO_IO1a: now also J3.5 (Pin_5); no longer J2.5 (Pin_5)
- net SAO_IO2 renamed SAO_IO2a
- net SAO_IO2a: now also J3.6 (Pin_6); no longer J2.6 (Pin_6)
- no-connect marks 0 -> 3
Other:
- moved on the sheet: J2
